Commit message: added FlipperCAD for left and right foot

File: urdf/atlas_v5.urdf (robot description, URDF)
Before this commit: robot drc_skeleton, 37 links, 36 joints
Links:
- link l_foot: geometry collision mesh filename=package://cs133a_project/meshes/FlipperCAD.STL; visual mesh filename=package://cs133a_project/meshes/FlipperCAD.STL
- link r_foot: geometry collision mesh filename=package://cs133a_project/meshes/FlipperCAD.STL; visual mesh filename=package://cs133a_project/meshes/FlipperCAD.STL

Commit message: Ball and robot at same time

File: urdf/atlas_v5.urdf (robot description, URDF)
Before this commit: robot drc_skeleton, 37 links, 36 joints
Links:
- link l_foot: geometry collision mesh filename=package://cs133a_project/meshes_unplugged/l_foot.dae; visual mesh filename=package://cs133a_project/meshes_unplugged/l_foot.dae
- link r_foot: geometry collision mesh filename=package://cs133a_project/meshes_unplugged/r_foot.dae; visual mesh filename=package://cs133a_project/meshes_unplugged/r_foot.dae
